File: hardware/mcu.kicad_sch (KiCad schematic)
At the start: 39 parts, among them J2 Conn_01x04, J3 Conn_01x02, J4 Conn_01x02, J5 Conn_01x01_Pin, J6 Conn_01x01_Pin, J7 Conn_01x01_Pin, SW1 SKRPACE010, U1 STM32G431KBUx, U2 DRV8311H, U3 AS5600L-ASOM, U5 TCAN330

Commit message: PCBをデイジーチェーンに対応
Parts:
- added J8: Conn_01x02, Connector_JST:JST_ZH_B2B-ZR_1x02_P1.50mm_Vertical, symbol Connector_Generic:Conn_01x02
Connections:
- net CAN_H: now also J8.1 (Pin_1)
- net CAN_L: now also J8.2 (Pin_2)
Changed lines of the file:
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@@
 	)
 	(junction
+		(at 41.91 167.64)
+		(diameter 0)
+		(color 0 0 0 0)
+	)
+	(junction
 		(at 92.71 34.29)
 		(diameter 0)
@@
 	)
 	(junction
+		(at 43.18 170.18)
+		(diameter 0)
+		(color 0 0 0 0)
+	)
+	(junction
 		(at 118.11 100.33)
 		(diameter 0)
@@
 	(wire
 		(pts
+			(xy 40.64 180.34) (xy 41.91 180.34)
+		)
+		(stroke
+			(width 0)
+			(type default)
+		)
+	)
+	(wire
+		(pts
 			(xy 194.31 100.33) (xy 196.85 100.33)
 		)
@@
 	(wire
 		(pts
-			(xy 40.64 170.18) (xy 45.72 170.18)
+			(xy 40.64 170.18) (xy 43.18 170.18)
 		)
 		(stroke
@@
 	(wire
 		(pts
+			(xy 43.18 182.88) (xy 43.18 170.18)
+		)
+		(stroke
+			(width 0)
+			(type default)
+		)
+	)
+	(wire
+		(pts
 			(xy 120.65 156.21) (xy 123.19 156.21)
 		)
@@
 	(wire
 		(pts
+			(xy 43.18 170.18) (xy 45.72 170.18)
+		)
+		(stroke
+			(width 0)
+			(type default)
+		)
+	)
+	(wire
+		(pts
 			(xy 209.55 127) (xy 209.55 129.54)
 		)
@@
 	(wire
 		(pts
+			(xy 41.91 180.34) (xy 41.91 167.64)
+		)
+		(stroke
+			(width 0)
+			(type default)
+		)
+	)
+	(wire
+		(pts
 			(xy 107.95 165.1) (xy 107.95 168.91)
 		)
@@
 	(wire
 		(pts
-			(xy 40.64 167.64) (xy 45.72 167.64)
+			(xy 40.64 167.64) (xy 41.91 167.64)
 		)
 		(stroke
@@
 	(wire
 		(pts
+			(xy 40.64 182.88) (xy 43.18 182.88)
+		)
+		(stroke
+			(width 0)
+			(type default)
+		)
+	)
+	(wire
+		(pts
 			(xy 212.09 85.09) (xy 212.09 73.66)
 		)
@@
 	(wire
 		(pts
+			(xy 41.91 167.64) (xy 45.72 167.64)
+		)
+		(stroke
+			(width 0)
+			(type default)
+		)
+	)
+	(wire
+		(pts
 			(xy 120.65 34.29) (xy 120.65 46.99)
 		)
@@
 					(unit 1)
 				)
+			)
+		)
+	)
+	(symbol
+		(lib_id "Connector_Generic:Conn_01x02")
+		(at 35.56 180.34 0)
+		(mirror y)
+		(unit 1)
+		(body_style 1)
+		(exclude_from_sim no)
+		(in_bom yes)
+		(on_board yes)
+		(in_pos_files yes)
+		(dnp no)
+		(fields_autoplaced yes)
+		(property "Reference" "J8"
+			(at 35.56 173.99 0)
+			(show_name no)
+			(do_not_autoplace no)
+			(effects
+				(font
+					(size 1.27 1.27)
+				)
+			)
+		)
+		(property "Value" "Conn_01x02"
+			(at 35.56 176.53 0)
+			(show_name no)
+			(do_not_autoplace no)
+			(effects
+				(font
+					(size 1.27 1.27)
+				)
+			)
+		)
+		(property "Footprint" "Connector_JST:JST_ZH_B2B-ZR_1x02_P1.50mm_Vertical"
+			(at 35.56 180.34 0)
+			(hide yes)
+			(show_name no)
+			(do_not_autoplace no)
+			(effects
+				(font
+					(size 1.27 1.27)
+				)
+			)
+		)
+		(property "Datasheet" ""
+			(at 35.56 180.34 0)
+			(hide yes)
+			(show_name no)
+			(do_not_autoplace no)
+			(effects
+				(font
+					(size 1.27 1.27)
+				)
+			)
+		)
+		(property "Description" "Generic connector, single row, 01x02, script generated (kicad-library-utils/schlib/autogen/connector/)"
+			(at 35.56 180.34 0)
+			(hide yes)
+			(show_name no)
+			(do_not_autoplace no)
+			(effects
+				(font
+					(size 1.27 1.27)
+				)
+			)
+		)
+		(pin "2"
+		)
+		(pin "1"
+		)
+		(instances
+			(project "hqdd_1"
+				(path "/c2b90e11-c7ad-42c4-9037-fc077dd1a3c2/7bbdb4b5-f615-4e52-82a7-d8572e7f02d6"
+					(reference "J8")
+					(unit 1)
+				)
