File: hardware/power.kicad_sch (KiCad schematic)
At the start: 16 parts, among them IC1 TAR5SB33, IC2 TAR5SB33, J1 Conn_01x02

Commit message: PCBをデイジーチェーンに対応
Parts:
- J1: footprint Connector_AMASS:AMASS_XT30U-M_1x02_P5.0mm_Vertical -> Connector_AMASS:AMASS_XT30UPB-M_1x02_P5.0mm_Vertical
Changed lines of the file:
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@@
 			)
 		)
-		(property "Footprint" "Connector_AMASS:AMASS_XT30U-M_1x02_P5.0mm_Vertical"
+		(property "Footprint" "Connector_AMASS:AMASS_XT30UPB-M_1x02_P5.0mm_Vertical"
 			(at 59.69 80.01 0)
 			(hide yes)
